File: torn_left/torn_left.kicad_pcb (KiCad board)
At the start: 2 copper layers, 140.7 x 115.6 mm, 76 parts, among them J1 SJ-43514, SW1 SW_Push, SW10 SW_Push, SW11 SW_Push, SW12 SW_Push, SW13 SW_Push, SW14 SW_Push, SW15 SW_Push, SW16 SW_Push, SW17 SW_Push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

Commit message: preparing for new board revision
Parts:
- removed R1: 1.5k, footprints:R_Axial_DIN0204_L3.6mm_D1.6mm_P5.08mm_Horizontal
- removed R4, R5: 5.1k, footprints:R_Axial_DIN0204_L3.6mm_D1.6mm_P5.08mm_Horizontal
- USB1: value USB_C_GCT_USB4085-Type-C -> USB_B_Mini; footprint footprints:USB_C_GCT_USB4085 -> footprints:USB-B-Mini-Right-Angled
- moved USB1 3.26 mm to (163.3, 55.9)
- moved H9 0.19 mm to (186.8, 54.2)
Connections:
- D50 pad 1: Net-(D50-Pad1) -> Net-(D50-K)
- D51 pad 1: Net-(D51-Pad1) -> Net-(D51-K)
- F1 pad 1: Net-(F1-Pad1) -> Net-(USB1-VBUS)
- R2 pad 2: Net-(D50-Pad1) -> Net-(D50-K)
- R3 pad 2: Net-(D51-Pad1) -> Net-(D51-K)
- U1 pad 21: Net-(U1-Pad21) -> unconnected-(U1-AREF-Pad21)
- U1 pad 23: Net-(U1-Pad23) -> unconnected-(U1-PC0-Pad23)
- U1 pad 24: Net-(U1-Pad24) -> unconnected-(U1-PC1-Pad24)
- U1 pad 25: Net-(U1-Pad25) -> unconnected-(U1-PC2-Pad25)
- U1 pad 26: Net-(U1-Pad26) -> unconnected-(U1-PC3-Pad26)
Routing:
- net Net-(D51-Pad1): track 54.4 -> 0.00 mm, vias 1 -> 0
- net Net-(D50-Pad1): track 53.3 -> 0.00 mm, vias 1 -> 0
- net Net-(D50-K): track 0.00 -> 37.4 mm, vias 0 -> 3
- net Net-(F1-Pad1): track 36.9 -> 0.00 mm
- net Net-(D51-K): track 0.00 -> 32.4 mm, vias 0 -> 2
- net Net-(USB1-VBUS): track 0.00 -> 23.5 mm, vias 0 -> 4
- net Net-(R4-Pad2): track 13.4 -> 0.00 mm, vias 1 -> 0
- net Net-(R5-Pad2): track 13.2 -> 0.00 mm
- net /COL0: track 164.1 -> 153.8 mm
- net /COL4: track 219.0 -> 211.2 mm
- net /ENC0_B: track 238.5 -> 232.9 mm, vias 3 -> 4
- net +5V: track 145.1 -> 139.8 mm
- net /i2c_SDA: track 83.0 -> 85.4 mm
- net /ROW3: track 155.4 -> 157.8 mm, vias 0 -> 1
- net Net-(D10-A): track 65.0 -> 63.1 mm
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Other:
- net class Default removed
- net class Power removed
- rule pad_to_mask_clearance: 0.2 -> 0.038

Commit message: committing before changing to standard size through hole resistors
Parts:
- added REF**: logo_42berlin, footprints:logo_42berlin, F.Cu at (56.8, 65.8)
Routing:
- net Net-(D50-K): track 37.4 -> 32.6 mm, vias 3 -> 1
- net Net-(USB1-VBUS): track 23.5 -> 19.1 mm, vias 4 -> 0
- net /ENC0_A: track 251.4 -> 254.1 mm
- net /ENC0_B: track 232.9 -> 235.4 mm
- net Net-(D51-K): track 32.4 -> 34.2 mm, vias 2 -> 1
- net /i2c_SDA: track 85.4 -> 84.5 mm
- net GND: track 8.08 -> 7.50 mm
- net Net-(D21-A): track 137.6 -> 137.1 mm
Other:
- board text added: "Torn Left rev 3.1"
- board text removed: "Torn Left rev 3.0"

Commit message: changed resistor sizes to more common 1/4W 0207DIN sizes on both boards
Parts:
- added R1: 1.5k, Resistor_THT:R_Axial_DIN0207_L6.3mm_D2.5mm_P7.62mm_Horizontal, F.Cu at (179.8, 85.6)
- R2, R3, R6, R7, R8: footprint footprints:R_Axial_DIN0204_L3.6mm_D1.6mm_P5.08mm_Horizontal -> Resistor_THT:R_Axial_DIN0207_L6.3mm_D2.5mm_P7.62mm_Horizontal
- moved R6 2.17 mm to (142.4, 60.6)
- moved R8 2.17 mm to (148.7, 60.6)
- moved R7 2.00 mm to (145.5, 60.6)
- moved D50 1.54 mm to (170.6, 79.2)
- moved D51 1.32 mm to (182.8, 79.2)
- moved R3 1.24 mm to (173.5, 85.6)
- moved C3 0.95 mm to (183.0, 73.0)
- moved R2 0.77 mm to (176.7, 85.6)
- moved F1 0.51 mm to (182.3, 67.2)
Routing:
- net +5V: track 139.8 -> 145.1 mm
- net Net-(D50-K): track 32.6 -> 35.3 mm
- net /i2c_SCL: track 73.5 -> 71.7 mm
- net /RESET: track 126.5 -> 128.1 mm
- net /i2c_SDA: track 84.5 -> 83.4 mm
Other:
- board text added: "Torn Left 42 edition rev 3.1"
- board text added: "Torn keyboard 42 edition licensed under CC BY-NC 4.0"
- board text added: "Torn keyboard licensed under CC BY-NC 4.0 42 edition"
- board text added: "https://github.com/fablabnk/torn"
- board text removed: "Torn Left rev 3.1"
- board text removed: "Torn keyboard licensed under CC BY-NC 4.0"
- board text removed: "https://github.com/rtitmuss/torn"
