File: torn_right/torn_right.kicad_sch (KiCad schematic)
At the start: 64 parts, among them J2 SJ-43514, J3 Conn_01x04, SW23 SW_Push, SW24 SW_Push, SW25 SW_Push, SW26 SW_Push, SW27 SW_Push, SW28 Rotary_Encoder_Switch, SW29 SW_Push, SW30 SW_Push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

Commit message: changed resistor sizes to more common 1/4W 0207DIN sizes on both boards
Parts:
- R50, R51, R52: footprint footprints:R_Axial_DIN0204_L3.6mm_D1.6mm_P5.08mm_Horizontal -> Resistor_THT:R_Axial_DIN0207_L6.3mm_D2.5mm_P7.62mm_Horizontal
Changed lines of the file:
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@@
 			)
 		)
-		(property "Footprint" "footprints:R_Axial_DIN0204_L3.6mm_D1.6mm_P5.08mm_Horizontal"
+		(property "Footprint" "Resistor_THT:R_Axial_DIN0207_L6.3mm_D2.5mm_P7.62mm_Horizontal"
 			(at 140.97 37.592 90)
 			(effects
@@
 			)
 		)
-		(property "Footprint" "footprints:R_Axial_DIN0204_L3.6mm_D1.6mm_P5.08mm_Horizontal"
+		(property "Footprint" "Resistor_THT:R_Axial_DIN0207_L6.3mm_D2.5mm_P7.62mm_Horizontal"
 			(at 140.97 47.752 90)
 			(effects
@@
 			)
 		)
-		(property "Footprint" "footprints:R_Axial_DIN0204_L3.6mm_D1.6mm_P5.08mm_Horizontal"
+		(property "Footprint" "Resistor_THT:R_Axial_DIN0207_L6.3mm_D2.5mm_P7.62mm_Horizontal"
 			(at 140.97 57.912 90)
 			(effects

Commit message: right board updated with proper TRRS and other fixes - reminder to check left side passes DRC
Parts:
- J2: footprint footprints:CUI_SJ-43514 -> footprints:PJ-320A
Changed lines of the file:
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@@
 			)
 		)
-		(property "Footprint" "footprints:CUI_SJ-43514"
+		(property "Footprint" "footprints:PJ-320A"
 			(at 92.71 114.3 0)
 			(effects
